Commit message: Expand camera's field of view.

File: urdf/turtlebot3_waffle_pi.urdf.xacro (robot description, xacro)
@@ -2,5 +2,5 @@
 <robot name="turtlebot3_waffle_pi" xmlns:xacro="http://ros.org/wiki/xacro">
   <xacro:include filename="$(find turtlebot3_description)/urdf/common_properties.xacro"/>
-  <xacro:include filename="$(find turtlebot3_description)/urdf/turtlebot3_waffle_pi.gazebo.xacro"/>
+  <xacro:include filename="$(find rob301_simulation)/urdf/turtlebot3_waffle_pi.gazebo.xacro"/>
   <link name="base_footprint"/>
   <joint name="base_joint" type="fixed">
@@ -164,5 +164,5 @@
     <!-- <origin xyz="0.073 -0.011 0.084" rpy="0 0 0"/> -->
     <!-- Down-facing camera, shifted forward so none of the robot itself is visible -->
-    <origin xyz="0.100 -0.011 0.084" rpy="0 1.57 0"/>
+    <origin xyz="0.120 -0.011 0.084" rpy="0 1.57 0"/>
     <parent link="base_link"/>
     <child link="camera_link"/>
